File: apoce board/apoce.kicad_sch (KiCad schematic)
At the start: 40 parts, among them J1 Test Soleil, J2 Solaire, J3 Test J/N, J4 Jour/Nuit, J5 Relais, SW1 ButModeJN, SW2 ButModeSol, SW3 ButModeAuto, SW4 ButArmV, U1 4N35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

Commit message: Revert "Nouvelle version avec amélioration"
This reverts commit 7894d477df82a93182f71be82a563ec3e50d3505.
Parts:
- D11: value LedModeSol-Orange -> LedModeSolCAV-Orange
- D12: value LedModeAuto-Rouge -> LedModeSolAuto-Rouge
- SW2: value ButModeSol -> ButModeSolCAV
- SW3: value ButModeAuto -> ButModeSolAuto
Changed lines of the file:
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@@
 			)
 		)
-		(property "Value" "ButModeSol"
+		(property "Value" "ButModeSolCAV"
 			(at 54.61 132.08 0)
 			(effects
@@
 			)
 		)
-		(property "Value" "LedModeSol-Orange"
+		(property "Value" "LedModeSolCAV-Orange"
 			(at 195.8975 129.54 0)
 			(effects
@@
 			)
 		)
-		(property "Value" "ButModeAuto"
+		(property "Value" "ButModeSolAuto"
 			(at 54.61 153.67 0)
 			(effects
@@
 			)
 		)
-		(property "Value" "LedModeAuto-Rouge"
+		(property "Value" "LedModeSolAuto-Rouge"
 			(at 195.8975 144.78 0)
 			(effects
